Commit message: add launch file for end_effector_withModel (UR5e without Moveit driver)

File: src/end_effector_description/urdf/end_effector_withModel.xacro (robot description, xacro)
@@ -1,12 +1,12 @@
 <?xml version="1.0" ?>
-<!-- Only displays the end-effector -->
-<robot name="end_effector_only" xmlns:xacro="http://ros.org/wiki/xacro">
+<!-- displays the end-effector with UR5e(no Moveit support)-->
+<robot name="end_effector_withModel" xmlns:xacro="http://ros.org/wiki/xacro">
   <!-- Including the claw.urdf.xacro file to give scope to xacro:claw. Inclusion is a simple copy-and-paste of code. -->
   <xacro:include filename="$(find end_effector_description)/urdf/end_effector.urdf.xacro" />
   <!-- UR5e robot arm -->
   <!-- URDF won't build if following args aren't defined. -->
-  <!-- <xacro:arg name="name" default="ur5"/>
+  <xacro:arg name="name" default="ur5"/>
   <xacro:arg name="ur_type" default="ur5"/>
-  <xacro:include filename="$(find ur_description)/urdf/ur.urdf.xacro"/> -->
+  <xacro:include filename="$(find ur_description)/urdf/ur.urdf.xacro"/>
   <!-- This is the abstract link which the base of the claw attaches to. -->
   <link name="end_effector_root_link"/>
@@ -17,7 +17,7 @@
   </xacro:end_effector>
   <!-- Coupler between arm and end effector -->
-  <!-- <joint name="ur5_end_effector_coupler_joint" type="fixed">
+  <joint name="ur5_end_effector_coupler_joint" type="fixed">
     <parent link="tool0"/>
-    <child link="end_effector_root_link"/> -->
-  <!-- </joint> -->
+    <child link="end_effector_root_link"/>
+  </joint>
 </robot>
