Commit message: add end_effector_only launch file, end_effector with robot still not working

File: src/end_effector_description/urdf/end_effector.urdf.xacro (robot description, xacro)
@@ -6,5 +6,5 @@
 <!-- The name of the robot is given here. xmlns:xacro is mandatory for xacro files. -->
 <robot name="end_effector" xmlns:xacro="http://ros.org/wiki/xacro">
-  <xacro:property name="scale_factor" value="0.002"/>
+  <xacro:property name="scale_factor" value="0.0015"/>
   <!--
     This is the start of a macro block called "claw".

File: src/end_effector_description/urdf/end_effector_only.xacro (robot description, xacro)
@@ -1,5 +1,5 @@
 <?xml version="1.0" ?>
 <!-- The purpose of this file is to fix the claw to some abstract link so the claw can be used in the world. -->
-<robot name="end_effector" xmlns:xacro="http://ros.org/wiki/xacro">
+<robot name="end_effector_only" xmlns:xacro="http://ros.org/wiki/xacro">
   <!-- Including the claw.urdf.xacro file to give scope to xacro:claw. Inclusion is a simple copy-and-paste of code. -->
   <xacro:include filename="$(find end_effector_description)/urdf/end_effector.urdf.xacro" />
@@ -17,7 +17,7 @@
   </xacro:end_effector>
   <!-- Coupler between arm and end effector -->
-  <joint name="ur5_end_effector_coupler_joint" type="fixed">
+  <!-- <joint name="ur5_end_effector_coupler_joint" type="fixed">
     <parent link="tool0"/>
-    <child link="end_effector_root_link"/>
-  </joint>
+    <child link="end_effector_root_link"/> -->
+  <!-- </joint> -->
 </robot>

Commit message: fake UR5e with driver support launch successfully, planning failed

File: src/end_effector_description/urdf/end_effector.urdf.xacro (robot description, xacro)
@@ -35,14 +35,4 @@
         <origin xyz="0 0 0" rpy="${pi} 0 ${pi}"/>
       </visual>
-      <!-- Defines the collision boundaries. -->
-      <collision>
-        <!-- Shape of object. -->
-        <geometry>
-          <mesh filename="package://end_effector_description/meshes/end_effector.stl" scale= "${scale_factor} ${scale_factor} ${scale_factor}"/>
-          <!-- <scale>${scale_factor} ${scale_factor} ${scale_factor}</scale> -->
-		</geometry>
-        <!-- Collision origin is usually the same as the visual origin. -->
-        <origin xyz="0 0 0" rpy="${pi} 0 ${pi}"/>
-      </collision>
       <!--
         Defines the inertial properties of the link.

Commit message: add dy_trans for camera_link

File: src/end_effector_description/urdf/end_effector.urdf.xacro (robot description, xacro)
@@ -49,4 +49,10 @@
       </inertial>
     </link>
+    <link name="${prefix}_camera_socket"> </link>
+    <joint name="${prefix}_camera_joint" type="fixed">
+        <parent link="${prefix}base_link"/>
+        <child link="${prefix}_camera_socket"/>
+        <origin xyz="0 0 0.1" rpy="0 0 0"/>
+    </joint>
   </xacro:macro>
 </robot>

File: src/end_effector_description/urdf/end_effector_only.xacro (robot description, xacro)
@@ -4,9 +4,4 @@
   <!-- Including the claw.urdf.xacro file to give scope to xacro:claw. Inclusion is a simple copy-and-paste of code. -->
   <xacro:include filename="$(find end_effector_description)/urdf/end_effector.urdf.xacro" />
-  <!-- UR5e robot arm -->
-  <!-- URDF won't build if following args aren't defined. -->
-  <!-- <xacro:arg name="name" default="ur5"/>
-  <xacro:arg name="ur_type" default="ur5"/>
-  <xacro:include filename="$(find ur_description)/urdf/ur.urdf.xacro"/> -->
   <!-- This is the abstract link which the base of the claw attaches to. -->
   <link name="end_effector_root_link"/>
@@ -16,8 +11,3 @@
     <origin xyz="0 0 0" rpy="0 0 0"/>
   </xacro:end_effector>
-  <!-- Coupler between arm and end effector -->
-  <!-- <joint name="ur5_end_effector_coupler_joint" type="fixed">
-    <parent link="tool0"/>
-    <child link="end_effector_root_link"/> -->
-  <!-- </joint> -->
 </robot>

Commit message: scale tuning, transformation tuning based on engineering drawing, update README

File: src/end_effector_description/urdf/end_effector.urdf.xacro (robot description, xacro)
@@ -6,5 +6,5 @@
 <!-- The name of the robot is given here. xmlns:xacro is mandatory for xacro files. -->
 <robot name="end_effector" xmlns:xacro="http://ros.org/wiki/xacro">
-  <xacro:property name="scale_factor" value="0.0015"/>
+  <xacro:property name="scale_factor" value="0.001"/>
   <!--
     This is the start of a macro block called "claw".
@@ -53,5 +53,5 @@
         <parent link="${prefix}base_link"/>
         <child link="${prefix}_camera_socket"/>
-        <origin xyz="0 0 0.1" rpy="0 0 0"/>
+        <origin xyz="0 0 0.07989" rpy="0 0 0"/>
     </joint>
   </xacro:macro>

Commit message: Merge david_addStaticLink; Add dy_trans for camera_link, update model scaling (#7)
* add dy_trans for camera_link

* scale tuning, transformation tuning based on engineering drawing, update README

File: src/end_effector_description/urdf/end_effector.urdf.xacro (robot description, xacro)
@@ -6,5 +6,5 @@
 <!-- The name of the robot is given here. xmlns:xacro is mandatory for xacro files. -->
 <robot name="end_effector" xmlns:xacro="http://ros.org/wiki/xacro">
-  <xacro:property name="scale_factor" value="0.0015"/>
+  <xacro:property name="scale_factor" value="0.001"/>
   <!--
     This is the start of a macro block called "claw".
@@ -49,4 +49,10 @@
       </inertial>
     </link>
+    <link name="${prefix}_camera_socket"> </link>
+    <joint name="${prefix}_camera_joint" type="fixed">
+        <parent link="${prefix}base_link"/>
+        <child link="${prefix}_camera_socket"/>
+        <origin xyz="0 0 0.07989" rpy="0 0 0"/>
+    </joint>
   </xacro:macro>
 </robot>

Commit message: fixing end_effector orientation

File: src/end_effector_description/urdf/end_effector.urdf.xacro (robot description, xacro)
@@ -33,5 +33,5 @@
 		</geometry>
         <!-- Origin of the visual element. xyz is in metres. rpy stands for roll pitch yaw in radians. -->
-        <origin xyz="0 0 0" rpy="${pi} 0 ${pi}"/>
+        <origin xyz="0 0 0" rpy="${pi} 0 ${pi/2}"/>
       </visual>
       <!-- Collision is removed for planning to work -->

Commit message: enable collosion check, add toolpoint_link and camera_link, deprecated transformation pkg

File: src/end_effector_description/urdf/end_effector.urdf.xacro (robot description, xacro)
@@ -7,4 +7,5 @@
 <robot name="end_effector" xmlns:xacro="http://ros.org/wiki/xacro">
   <xacro:property name="scale_factor" value="0.001"/>
+  <xacro:property name="end_effector_displacement" value="0.04"/>
   <!--
     This is the start of a macro block called "claw".
@@ -15,11 +16,10 @@
     * denotes that the variable is a tag. Literally <origin xyz=... />
   -->
-  <xacro:macro name="end_effector" params="prefix parent *origin">
+  <xacro:macro name="end_effector" params="prefix parent">
     <!-- This joint fixes the claw to an external parent link (could be the world or another robot). -->
     <joint name="${prefix}end_effector_flange" type="fixed">
       <parent link="${parent}"/>
       <child link="${prefix}base_link"/>
-      <!-- xacro:insert_block means place the tag here. Specify the positional relationship between parent and child links. -->
-      <xacro:insert_block name="origin"/>
+      <origin xyz="0 0 0.04" rpy="0 0 0"/>
     </joint>
     <!-- Define a link for mesh base_link.STL. -->
@@ -28,12 +28,18 @@
       <visual>
         <!-- Shape of object. -->
-        <geometry>
+      <geometry>
           <mesh filename="package://end_effector_description/meshes/end_effector.stl" scale= "${scale_factor} ${scale_factor} ${scale_factor}"/>
 		  <!-- <scale>${scale_factor} ${scale_factor} ${scale_factor}</scale> -->
-		</geometry>
+      </geometry>
         <!-- Origin of the visual element. xyz is in metres. rpy stands for roll pitch yaw in radians. -->
-        <origin xyz="0 0 0" rpy="${pi} 0 ${pi}"/>
+        <origin xyz="0 0 0" rpy="${pi} 0 ${pi/2}"/>
       </visual>
-      <!-- Collision is removed for planning to work -->
+      <!-- Collision properties -->
+      <collision>
+        <geometry>
+          <mesh filename="package://end_effector_description/meshes/end_effector.stl" scale="${scale_factor} ${scale_factor} ${scale_factor}"/>
+        </geometry>
+        <origin xyz="0 0 0" rpy="${pi} 0 ${pi/2}"/>
+      </collision>
       <!--
         Defines the inertial properties of the link.
@@ -49,9 +55,15 @@
       </inertial>
     </link>
-    <link name="${prefix}_camera_socket"> </link>
+    <link name="camera_link"> </link>
     <joint name="${prefix}_camera_joint" type="fixed">
         <parent link="${prefix}base_link"/>
-        <child link="${prefix}_camera_socket"/>
-        <origin xyz="0 0 0.07989" rpy="0 0 0"/>
+        <child link="camera_link"/>
+        <origin xyz="-0.02 0 0.07989" rpy="0 0 0"/>
+    </joint>
+    <link name="${prefix}_tool_point"> </link>
+    <joint name="${prefix}_tool_point_joint" type="fixed">
+        <parent link="${prefix}base_link"/>
+        <child link="${prefix}_tool_point"/>
+        <origin xyz="-0.0975 0 0.02" rpy="0 0 0"/>
     </joint>
   </xacro:macro>

File: src/end_effector_description/urdf/end_effector_only.xacro (robot description, xacro)
@@ -8,6 +8,4 @@
   <!-- Instantiate the claw by using its macro. -->
   <xacro:end_effector prefix="4231" parent="end_effector_root_link" >
-    <!-- Note that we are passing in a tag as an argument. -->
-    <origin xyz="0 0 0" rpy="0 0 0"/>
   </xacro:end_effector>
 </robot>

File: src/end_effector_description/urdf/end_effector_withDriverSupport.xacro (robot description, xacro)
@@ -13,6 +13,4 @@
   <!-- Instantiate the claw by using its macro. -->
   <xacro:end_effector prefix="4231" parent="end_effector_root_link" >
-    <!-- Note that we are passing in a tag as an argument. -->
-    <origin xyz="0 0 0" rpy="0 0 0"/>
   </xacro:end_effector>
   <!-- Coupler between arm and end effector -->

File: src/end_effector_description/urdf/end_effector_withModel.xacro (robot description, xacro)
@@ -13,6 +13,4 @@
   <!-- Instantiate the claw by using its macro. -->
   <xacro:end_effector prefix="4231" parent="end_effector_root_link" >
-    <!-- Note that we are passing in a tag as an argument. -->
-    <origin xyz="0 0 0" rpy="0 0 0"/>
   </xacro:end_effector>
   <!-- Coupler between arm and end effector -->

Commit message: Add collision detection, take into account housing and screwblock (4cm thickness), add toolpoint link and camera_link, deprecate tranformation pkg (#9)
* visualisation of housing and screwblock

* enable collosion check, add toolpoint_link and camera_link, deprecated transformation pkg

File: src/end_effector_description/urdf/end_effector.urdf.xacro (robot description, xacro)
@@ -7,4 +7,5 @@
 <robot name="end_effector" xmlns:xacro="http://ros.org/wiki/xacro">
   <xacro:property name="scale_factor" value="0.001"/>
+  <xacro:property name="end_effector_displacement" value="0.04"/>
   <!--
     This is the start of a macro block called "claw".
@@ -15,11 +16,10 @@
     * denotes that the variable is a tag. Literally <origin xyz=... />
   -->
-  <xacro:macro name="end_effector" params="prefix parent *origin">
+  <xacro:macro name="end_effector" params="prefix parent">
     <!-- This joint fixes the claw to an external parent link (could be the world or another robot). -->
     <joint name="${prefix}end_effector_flange" type="fixed">
       <parent link="${parent}"/>
       <child link="${prefix}base_link"/>
-      <!-- xacro:insert_block means place the tag here. Specify the positional relationship between parent and child links. -->
-      <xacro:insert_block name="origin"/>
+      <origin xyz="0 0 0.04" rpy="0 0 0"/>
     </joint>
     <!-- Define a link for mesh base_link.STL. -->
@@ -28,12 +28,18 @@
       <visual>
         <!-- Shape of object. -->
-        <geometry>
+      <geometry>
           <mesh filename="package://end_effector_description/meshes/end_effector.stl" scale= "${scale_factor} ${scale_factor} ${scale_factor}"/>
 		  <!-- <scale>${scale_factor} ${scale_factor} ${scale_factor}</scale> -->
-		</geometry>
+      </geometry>
         <!-- Origin of the visual element. xyz is in metres. rpy stands for roll pitch yaw in radians. -->
         <origin xyz="0 0 0" rpy="${pi} 0 ${pi/2}"/>
       </visual>
-      <!-- Collision is removed for planning to work -->
+      <!-- Collision properties -->
+      <collision>
+        <geometry>
+          <mesh filename="package://end_effector_description/meshes/end_effector.stl" scale="${scale_factor} ${scale_factor} ${scale_factor}"/>
+        </geometry>
+        <origin xyz="0 0 0" rpy="${pi} 0 ${pi/2}"/>
+      </collision>
       <!--
         Defines the inertial properties of the link.
@@ -49,9 +55,15 @@
       </inertial>
     </link>
-    <link name="${prefix}_camera_socket"> </link>
+    <link name="camera_link"> </link>
     <joint name="${prefix}_camera_joint" type="fixed">
         <parent link="${prefix}base_link"/>
-        <child link="${prefix}_camera_socket"/>
-        <origin xyz="0 0 0.07989" rpy="0 0 0"/>
+        <child link="camera_link"/>
+        <origin xyz="-0.02 0 0.07989" rpy="0 0 0"/>
+    </joint>
+    <link name="${prefix}_tool_point"> </link>
+    <joint name="${prefix}_tool_point_joint" type="fixed">
+        <parent link="${prefix}base_link"/>
+        <child link="${prefix}_tool_point"/>
+        <origin xyz="-0.0975 0 0.02" rpy="0 0 0"/>
     </joint>
   </xacro:macro>

Commit message: critical fix to transformation urdf frame rotation

File: src/end_effector_description/urdf/end_effector.urdf.xacro (robot description, xacro)
@@ -59,5 +59,5 @@
         <parent link="${prefix}base_link"/>
         <child link="camera_link"/>
-        <origin xyz="-0.02 0 0.07989" rpy="0 0 0"/>
+        <origin xyz="-0.02 0 0.07989" rpy="${pi} ${pi} 0"/>
     </joint>
     <link name="${prefix}_tool_point"> </link>

Commit message: tune transformation

File: src/end_effector_description/urdf/end_effector.urdf.xacro (robot description, xacro)
@@ -21,5 +21,5 @@
       <parent link="${parent}"/>
       <child link="${prefix}base_link"/>
-      <origin xyz="0 0 0.04" rpy="0 0 0"/>
+      <origin xyz="0 0 0.01" rpy="0 0 0"/>
     </joint>
     <!-- Define a link for mesh base_link.STL. -->

Commit message: Move to screw fully working, change home position, change in arm-movement pkg, ignore large screws (#14)
* add centre detection algo, intermediate

* critical fix to transformation urdf frame rotation

* tune transformation

* fix concurrency issue, add stright-to-hole method

* intemediate save, tuning transformation for new home pos

* fully working, major milestone

* fixed vision to ignore the larger holes

File: src/end_effector_description/urdf/end_effector.urdf.xacro (robot description, xacro)
@@ -21,5 +21,5 @@
       <parent link="${parent}"/>
       <child link="${prefix}base_link"/>
-      <origin xyz="0 0 0.04" rpy="0 0 0"/>
+      <origin xyz="0 0 0.01" rpy="0 0 0"/>
     </joint>
     <!-- Define a link for mesh base_link.STL. -->
@@ -59,5 +59,5 @@
         <parent link="${prefix}base_link"/>
         <child link="camera_link"/>
-        <origin xyz="-0.02 0 0.07989" rpy="0 0 0"/>
+        <origin xyz="-0.02 0 0.07989" rpy="${pi} ${pi} 0"/>
     </joint>
     <link name="${prefix}_tool_point"> </link>
